Commit message: moved files around
what to only make one package, igvc25

File: src/igvc25/description/0_robot.urdf.xacro (robot description, xacro)
@@ -5,5 +5,5 @@
 <robot xmlns:xacro="http://www.ros.org/wiki/xacro"  name="robot">
     <!-- commandline args to determine how to build robot -->
-    <xacro:arg name="target_robot" default="test" />
+    <xacro:arg name="target_robot" default="fwd_c" />
     <!-- Origin of the robot in space - should be at pivot point
          basically a xyz origin reference with no shape or size -->
@@ -11,14 +11,9 @@
     <!-- Projection of base_link onto ground -->
     <link name="base_footprint"></link>
-    <joint name="footprint_joint" type="fixed">
-        <parent link="base_link"/>
-        <child link="base_footprint"/>
-        <!-- difference in pos of base link and footprint -->
-        <origin xyz="0.0 0.0 -1.0" rpy="0.0 0.0 0.0"/>
-    </joint>
     <!-- rviz2 materials -->
     <xacro:include filename="materials.xacro"/>
-    <!-- macros to generate inertial matrix -->
+    <!-- macros to generate common sections -->
     <xacro:include filename="inertial_macros.xacro"/>
+    <xacro:include filename="componet_macros.xacro"/>
     <!-- include selected robot description -->
     <xacro:include filename="$(arg target_robot)-robot/0_core.xacro"/>

File: src/igvc25/description/test-robot/0_core.xacro (robot description, xacro)
@@ -1,4 +1,10 @@
 <?xml version="1.0"?>
 <robot xmlns:xacro="http://www.ros.org/wiki/xacro"  name="robot">
+    <joint name="footprint_joint" type="fixed">
+        <parent link="base_link"/>
+        <child link="base_footprint"/>
+        <!-- difference in pos of base link and footprint -->
+        <origin xyz="0.0 0.0 -1.0" rpy="0.0 0.0 0.0"/>
+    </joint>
     <link name="test_link">
         <visual name="">

Commit message: lidar sim
meshes do not work though

File: src/igvc25/description/0_robot.urdf.xacro (robot description, xacro)
@@ -3,5 +3,5 @@
      for Ros2, Rviz2, and Gazebo-Classic
      It uses XACRO to break the single xml file into smaller more editable chunks -->
-<robot xmlns:xacro="http://www.ros.org/wiki/xacro"  name="robot">
+<robot xmlns:xacro="http://www.ros.org/wiki/xacro"  name="sarah">
     <!-- commandline args to determine how to build robot -->
     <xacro:arg name="target_robot" default="test" />
@@ -17,5 +17,9 @@
     <xacro:include filename="macros/inertial_macros.xacro"/>
     <xacro:include filename="macros/componet_macros.xacro"/>
+    <xacro:include filename="macros/vlp16.xacro"/>
     <!-- include selected robot description -->
     <xacro:include filename="$(arg target_robot).robot.xacro"/>
+     <xacro:VLP-16 parent="base_link">
+          <origin xyz="0 0 1" rpy="0 0 0" />
+     </xacro:VLP-16>
 </robot>

Commit message: ros-gz-bridge working
can get sensor data from sim, and send control input to sim, yay!

File: src/igvc25/description/0_robot.urdf.xacro (robot description, xacro)
@@ -5,6 +5,8 @@
 <robot xmlns:xacro="http://www.ros.org/wiki/xacro"  name="sarah">
     <!-- commandline args to determine how to build robot -->
-    <xacro:arg name="target_robot" default="test" />
-    <xacro:arg name="simulation"   default="true" />
+    <xacro:arg name="target_robot" default="test"/>
+    <xacro:arg name="simulation"   default="true"/>
+    <!-- properties -->
+    <xacro:property name="mesh_folder" value="/home/es/Documents/GitHub/IGVC25/src/igvc25/description/meshes"/>
     <!-- Origin of the robot in space - should be at pivot point
          basically a xyz origin reference with no shape or size -->
@@ -17,9 +19,8 @@
     <xacro:include filename="macros/inertial_macros.xacro"/>
     <xacro:include filename="macros/componet_macros.xacro"/>
-    <xacro:include filename="macros/vlp16.xacro"/>
     <!-- include selected robot description -->
     <xacro:include filename="$(arg target_robot).robot.xacro"/>
      <xacro:VLP-16 parent="base_link">
-          <origin xyz="0 0 1" rpy="0 0 0" />
+          <origin xyz="0 0 0.3" rpy="0 0 0"/>
      </xacro:VLP-16>
 </robot>

File: src/igvc25/description/fwd.robot.xacro (robot description, xacro)
@@ -86,10 +86,63 @@
         MARK: Control
     -->
-    <xacro:if value="$(arg simulation)"  >
-        <xacro:include filename="gz_control.xacro"/>
+    <xacro:unless value="$(arg simulation)">
+        <ros2_control name="RealRobot" type="system">
+            <hardware>
+                <plugin>diffdrive_arduino/DiffDriveArduinoHardware</plugin>
+                <param name="left_wheel_name">left_wheel_joint</param>
+                <param name="right_wheel_name">right_wheel_joint</param>
+                <param name="loop_rate">30</param>
+                <param name="device">/dev/ttyUSB0</param>
+                <param name="baud_rate">57600</param>
+                <param name="timeout_ms">1000</param>
+                <param name="enc_counts_per_rev">3436</param>
+            </hardware>
+            <joint name="left_wheel_joint">
+                <command_interface name="velocity">
+                    <param name="min">-10</param>
+                    <param name="max">10</param>
+                </command_interface>
+                <state_interface name="position"/>
+                <state_interface name="velocity"/>
+            </joint>
+            <joint name="right_wheel_joint">
+                <command_interface name="velocity">
+                    <param name="min">-10</param>
+                    <param name="max">10</param>
+                </command_interface>
+                <state_interface name="position"/>
+                <state_interface name="velocity"/>
+            </joint>
+        </ros2_control>
+    </xacro:unless>
+    <xacro:if value="$(arg simulation)">
+        <ros2_control name="GazeboSystem" type="system">
+            <hardware>
+                <plugin>gz_ros2_control/GazeboSimSystem</plugin>
+            </hardware>
+            <joint name="left_wheel_joint">
+                <command_interface name="velocity">
+                    <param name="min">-10</param>
+                    <param name="max">10</param>
+                </command_interface>
+                <state_interface name="velocity"/>
+                <state_interface name="position"/>
+            </joint>
+            <joint name="right_wheel_joint">
+                <command_interface name="velocity">
+                    <param name="min">-10</param>
+                    <param name="max">10</param>
+                </command_interface>
+                <state_interface name="velocity"/>
+                <state_interface name="position"/>
+            </joint>
+        </ros2_control>
     </xacro:if>
-    <xacro:unless value="$(arg simulation)"  >
-        <xacro:include filename="r2_control.xacro"/>
-    </xacro:unless>
+    <gazebo>
+        <plugin name="gz_ros2_control::GazeboSimROS2ControlPlugin" filename="libgz_ros2_control-system.so">
+            <parameters>$(find igvc25)/config/controllers.yaml</parameters>
+            <parameters>$(find igvc25)/config/controllers_sim.yaml</parameters>
+        </plugin>
+    </gazebo>
     <!--
         MARK: Sim

File: src/igvc25/description/macros/componet_macros.xacro (robot description, xacro)
@@ -1,4 +1,7 @@
 <?xml version="1.0"?>
 <robot xmlns:xacro="http://www.ros.org/wiki/xacro" >
+    <!--
+        MARK: wheel
+    -->
     <xacro:macro name="wheel" params="name parent_link wheel_distance wheel_radius wheel_length wheel_mass">
         <joint name="${name}_joint" type="continuous">
@@ -25,3 +28,103 @@
         </link>
     </xacro:macro>
+    <!--
+        MARK: lidar
+        -->
+    <xacro:macro name="VLP-16" params="*origin parent">
+        <!-- VLP-16 LiDAR -->
+        <joint name="velodyne_base_mount_joint" type="fixed">
+            <xacro:insert_block name="origin" />
+            <parent link="${parent}"/>
+            <child link="velodyne_base_link"/>
+        </joint>
+        <link name="velodyne_base_link">
+            <inertial>
+                <mass value="0.83"/>
+                <origin xyz="0 0 0.03585"/>
+                <inertia ixx="${(0.83 * (3.0*0.0516*0.0516 + 0.0717*0.0717)) / 12.0}" ixy="0" ixz="0"
+                iyy="${(0.83 * (3.0*0.0516*0.0516 + 0.0717*0.0717)) / 12.0}" iyz="0"
+                izz="${0.5 * 0.83 * (0.0516*0.0516)}"/>
+            </inertial>
+            <visual>
+                <!-- <geometry>
+                    <mesh filename="${mesh_folder}/VLP16_base_1.dae"/>
+                </geometry> -->
+                <geometry>
+                    <cylinder radius="${0.103 / 2.0}" length="0.072"/>
+                </geometry>
+                <material name="black"/>
+            </visual>
+            <!-- <visual>
+                <geometry>
+                    <mesh filename="${mesh_folder}/VLP16_base_2.dae"/>
+                </geometry>
+            </visual> -->
+            <collision>
+                <origin rpy="0 0 0" xyz="0 0 0.03585"/>
+                <geometry>
+                    <cylinder radius="0.0516" length="0.0717"/>
+                </geometry>
+            </collision>
+        </link>
+        <joint name="velodyne_base_scan_joint" type="fixed" >
+            <origin xyz="0 0 0.0377" rpy="0 0 0" />
+            <parent link="velodyne_base_link" />
+            <child link="velodyne"/>
+        </joint>
+        <link name="velodyne">
+            <inertial>
+                <mass value="0.01"/>
+                <origin xyz="0 0 0"/>
+                <inertia ixx="1e-7" ixy="0" ixz="0" iyy="1e-7" iyz="0" izz="1e-7"/>
+            </inertial>
+            <!-- <visual>
+                <origin xyz="0 0 -0.0377"/>
+                <geometry>
+                    <mesh filename="${mesh_folder}/VLP16_scan.dae"/>
+                </geometry>
+            </visual> -->
+            <collision>
+                <geometry>
+                    <sphere radius="0"/>
+                </geometry>
+            </collision>
+        </link>
+        <!-- Gazebo requires ... -->
+        <gazebo reference="velodyne">
+            <sensor name="velodyne" type="gpu_lidar">
+                <pose>0 0 0 0 0 0</pose>
+                <update_rate>10</update_rate>
+                <visualize>true</visualize>
+                <topic>velodyne_points</topic>
+                <always_on>true</always_on>
+                <gz_frame_id>velodyne</gz_frame_id>
+                <ray>
+                    <scan>
+                        <horizontal>
+                            <samples>1800</samples>
+                            <resolution>1</resolution>
+                            <min_angle>-3.14159</min_angle>
+                            <max_angle>3.14159</max_angle>
+                        </horizontal>
+                        <vertical>
+                            <samples>16</samples>
+                            <resolution>1</resolution>
+                            <min_angle>-0.261799</min_angle> <!-- -15 degrees -->
+                            <max_angle>0.261799</max_angle>  <!-- +15 degrees -->
+                        </vertical>
+                    </scan>
+                    <range>
+                        <min>0.1</min>
+                        <max>100.0</max>
+                        <resolution>0.01</resolution>
+                    </range>
+                    <noise>
+                        <type>gaussian</type>
+                        <mean>0.0</mean>
+                        <stddev>0.01</stddev>
+                    </noise>
+                </ray>
+            </sensor>
+        </gazebo>
+    </xacro:macro>
 </robot>

Commit message: imu sim working

File: src/igvc25/description/0_robot.urdf.xacro (robot description, xacro)
@@ -21,6 +21,3 @@
     <!-- include selected robot description -->
     <xacro:include filename="$(arg target_robot).robot.xacro"/>
-     <xacro:VLP-16 parent="base_link">
-          <origin xyz="0 0 0.3" rpy="0 0 0"/>
-     </xacro:VLP-16>
 </robot>

File: src/igvc25/description/fwd.robot.xacro (robot description, xacro)
@@ -84,4 +84,19 @@
     </link>
     <!--
+        MARK: Sensors
+    -->
+    <!-- Lidar -->
+     <xacro:VLP-16 parent="base_link">
+          <origin xyz="-0.3 0 0.5" rpy="0 0 0"/>
+     </xacro:VLP-16>
+    <!-- IMU -->
+     <xacro:ph-imu parent="velodyne">
+          <origin xyz="0 0 0.05" rpy="0 0 0"/>
+     </xacro:ph-imu>
+    <!-- GPS -->
+     <xacro:garmin-gps parent="imu">
+          <origin xyz="0 0 0.05" rpy="0 0 0"/>
+     </xacro:garmin-gps>
+    <!--
         MARK: Control
     -->

File: src/igvc25/description/macros/componet_macros.xacro (robot description, xacro)
@@ -30,7 +30,8 @@
     <!--
         MARK: lidar
-        -->
+    -->
     <xacro:macro name="VLP-16" params="*origin parent">
         <!-- VLP-16 LiDAR -->
+        <!-- meshes seems to be broken, using simple geometry instead -->
         <joint name="velodyne_base_mount_joint" type="fixed">
             <xacro:insert_block name="origin" />
@@ -128,3 +129,66 @@
         </gazebo>
     </xacro:macro>
+    <!--
+        MARK: imu
+    -->
+    <!-- Based on: https://www.phidgets.com/productfiles/MOT0110/MOT0110_0/Documentation/MOT0110_0_Mechanical.pdf -->
+    <xacro:macro name="ph-imu" params="*origin parent">
+        <joint name="imu_joint" type="fixed">
+            <parent link="${parent}"/>
+            <child link="imu"/>
+            <xacro:insert_block name="origin" />
+        </joint>
+        <link name="imu">
+            <visual>
+                <geometry>
+                    <box size="0.038989 0.037846 0.013380"/>
+                </geometry>
+                <material name="orange" />
+            </visual>
+        </link>
+        <gazebo reference="imu">
+            <sensor name="imu" type="imu">
+                <pose>0 0 0 0 0 0</pose>
+                <always_on>true</always_on>
+                <update_rate>1</update_rate>
+                <visualize>true</visualize>
+                <topic>imu</topic>
+                <gz_frame_id>imu</gz_frame_id>
+                <plugin filename="gz-sim-imu-system" name="gz::sim::systems::Imu">
+                </plugin>
+            </sensor>
+        </gazebo>
+    </xacro:macro>
+    <!--
+        MARK: GPS
+    -->
+    <!-- https://www.garmin.com/en-US/p/27594#overview -->
+    <xacro:macro name="garmin-gps" params="*origin parent">
+        <joint name="gps_joint" type="fixed">
+            <parent link="${parent}"/>
+            <child link="gps"/>
+            <xacro:insert_block name="origin" />
+        </joint>
+        <link name="gps">
+            <visual>
+                <geometry>
+                    <cylinder radius="0.0305" length="0.0195"/>
+                </geometry>
+                <material name="orange" />
+            </visual>
+        </link>
+        <gazebo reference="gps">
+            <sensor name="gps" type="navsat">
+                <pose>0 0 0 0 0 0</pose>
+                <always_on>true</always_on>
+                <update_rate>1</update_rate>
+                <visualize>true</visualize>
+                <topic>gps</topic>
+                <gz_frame_id>gps</gz_frame_id>
+                <plugin filename="gz-sim-gps-system"
+                    name="gz::sim::systems::Gps">
+                </plugin>
+            </sensor>
+        </gazebo>
+    </xacro:macro>
 </robot>
