Commit message: all sensors simulated

File: src/igvc25/description/fwd.robot.xacro (robot description, xacro)
@@ -87,15 +87,22 @@
     -->
     <!-- Lidar -->
-     <xacro:VLP-16 parent="base_link">
-          <origin xyz="-0.3 0 0.5" rpy="0 0 0"/>
-     </xacro:VLP-16>
+    <xacro:VLP-16 parent="base_link">
+        <origin xyz="-0.3 0 0.5" rpy="0 0 0"/>
+    </xacro:VLP-16>
     <!-- IMU -->
-     <xacro:ph-imu parent="velodyne">
-          <origin xyz="0 0 0.05" rpy="0 0 0"/>
-     </xacro:ph-imu>
+    <xacro:ph-imu parent="velodyne">
+        <origin xyz="0 0 0.05" rpy="0 0 0"/>
+    </xacro:ph-imu>
     <!-- GPS -->
-     <xacro:garmin-gps parent="imu">
-          <origin xyz="0 0 0.05" rpy="0 0 0"/>
-     </xacro:garmin-gps>
+    <xacro:garmin-gps parent="imu">
+        <origin xyz="0 0 0.05" rpy="0 0 0"/>
+    </xacro:garmin-gps>
+    <!-- Camera -->
+    <xacro:logi-cam parent="chassis_link" name="left_camera">
+        <origin xyz="0.5 ${wheel_distance} 0.05" rpy="0.0 0.0 0.523599"/>
+    </xacro:logi-cam>
+    <xacro:logi-cam parent="chassis_link" name="right_camera">
+        <origin xyz="0.5 -${wheel_distance} 0.05" rpy="0.0 0.0 -0.523599"/>
+    </xacro:logi-cam>
     <!--
         MARK: Control

File: src/igvc25/description/macros/componet_macros.xacro (robot description, xacro)
@@ -132,10 +132,10 @@
         MARK: imu
     -->
-    <!-- Based on: https://www.phidgets.com/productfiles/MOT0110/MOT0110_0/Documentation/MOT0110_0_Mechanical.pdf -->
+    <!-- https://www.phidgets.com/productfiles/MOT0110/MOT0110_0/Documentation/MOT0110_0_Mechanical.pdf -->
     <xacro:macro name="ph-imu" params="*origin parent">
         <joint name="imu_joint" type="fixed">
             <parent link="${parent}"/>
             <child link="imu"/>
-            <xacro:insert_block name="origin" />
+            <xacro:insert_block name="origin"/>
         </joint>
         <link name="imu">
@@ -144,5 +144,5 @@
                     <box size="0.038989 0.037846 0.013380"/>
                 </geometry>
-                <material name="orange" />
+                <material name="orange"/>
             </visual>
         </link>
@@ -155,5 +155,7 @@
                 <topic>imu</topic>
                 <gz_frame_id>imu</gz_frame_id>
-                <plugin filename="gz-sim-imu-system" name="gz::sim::systems::Imu">
+                <plugin
+                    filename="gz-sim-imu-system"
+                    name="gz::sim::systems::Imu">
                 </plugin>
             </sensor>
@@ -168,5 +170,5 @@
             <parent link="${parent}"/>
             <child link="gps"/>
-            <xacro:insert_block name="origin" />
+            <xacro:insert_block name="origin"/>
         </joint>
         <link name="gps">
@@ -175,5 +177,5 @@
                     <cylinder radius="0.0305" length="0.0195"/>
                 </geometry>
-                <material name="orange" />
+                <material name="orange"/>
             </visual>
         </link>
@@ -186,9 +188,57 @@
                 <topic>gps</topic>
                 <gz_frame_id>gps</gz_frame_id>
-                <plugin filename="gz-sim-gps-system"
-                    name="gz::sim::systems::Gps">
+                <plugin
+                    filename="gz-sim-navsat-system"
+                    name="gz::sim::systems::NavSat">
                 </plugin>
             </sensor>
         </gazebo>
     </xacro:macro>
+    <!--
+        MARK: Camera
+    -->
+    <!-- https://www.logitech.com/en-us/shop/p/c920s-pro-hd-webcam.960-001257 -->
+    <xacro:macro name="logi-cam" params="*origin name parent">
+        <joint name="${name}_joint" type="fixed">
+            <parent link="${parent}"/>
+            <child link="${name}_link"/>
+            <xacro:insert_block name="origin"/>
+        </joint>
+        <link name="${name}_link">
+            <visual>
+                <geometry>
+                    <box size="0.07112 0.09398 0.04318"/>
+                </geometry>
+                <material name="red"/>
+            </visual>
+        </link>
+        <joint name="${name}_optical_joint" type="fixed">
+            <parent link="${name}_link"/>
+            <child link="${name}_link_optical"/>
+            <origin xyz="0.03556 0 0" rpy="${-pi/2} 0 ${-pi/2}"/>
+        </joint>
+        <link name="${name}_link_optical"></link>
+        <gazebo reference="${name}_link">
+            <sensor name="${name}_camera" type="camera">
+                <pose> 0 0 0 0 0 0 </pose>
+                <visualize>true</visualize>
+                <update_rate>30</update_rate>
+                <camera>
+                    <camera_info_topic>${name}/camera_info</camera_info_topic>
+                    <horizontal_fov>1.2290609</horizontal_fov>
+                    <image>
+                        <format>R8G8B8</format>
+                        <width>1920</width>
+                        <height>1080</height>
+                    </image>
+                    <clip>
+                        <near>0.05</near>
+                        <far>8.0</far>
+                    </clip>
+                </camera>
+                <topic>${name}/image_raw</topic>
+                <gz_frame_id>${name}_link_optical</gz_frame_id>
+            </sensor>
+        </gazebo>
+    </xacro:macro>
 </robot>

Commit message: nav2 randomly stops
working through nav stack, also robot drives very slow

File: src/igvc25/description/fwd.robot.xacro (robot description, xacro)
@@ -87,9 +87,9 @@
     -->
     <!-- Lidar -->
-    <xacro:VLP-16 parent="base_link">
-        <origin xyz="-0.3 0 0.5" rpy="0 0 0"/>
-    </xacro:VLP-16>
+    <xacro:lidar parent="base_link">
+        <origin xyz="-0.3 0 0.3" rpy="0 0 0"/>
+    </xacro:lidar>
     <!-- IMU -->
-    <xacro:ph-imu parent="velodyne">
+    <xacro:ph-imu parent="lidar_frame">
         <origin xyz="0 0 0.05" rpy="0 0 0"/>
     </xacro:ph-imu>

File: src/igvc25/description/macros/componet_macros.xacro (robot description, xacro)
@@ -29,5 +29,45 @@
     </xacro:macro>
     <!--
-        MARK: lidar
+        MARK: flat-lidar
+    -->
+    <xacro:macro name="lidar" params="*origin parent">
+        <joint name="lidar_joint" type="fixed">
+            <parent link="${parent}"/>
+            <child link="lidar_frame"/>
+            <xacro:insert_block name="origin"/>
+        </joint>
+        <link name="lidar_frame">
+            <visual>
+                <geometry>
+                    <cylinder radius="0.05" length="0.04"/>
+                </geometry>
+                <material name="black"/>
+            </visual>
+        </link>
+        <gazebo reference="lidar_frame">
+            <sensor name="laser" type="gpu_lidar">
+                <pose> 0 0 0 0 0 0 </pose>
+                <visualize>false</visualize>
+                <update_rate>10</update_rate>
+                <lidar>
+                    <scan>
+                        <horizontal>
+                            <samples>360</samples>
+                            <min_angle>-3.14</min_angle>
+                            <max_angle>3.14</max_angle>
+                        </horizontal>
+                    </scan>
+                    <range>
+                        <min>0.3</min>
+                        <max>12</max>
+                    </range>
+                </lidar>
+                <topic>scan</topic>
+                <gz_frame_id>lidar_frame</gz_frame_id>
+            </sensor>
+        </gazebo>
+    </xacro:macro>
+    <!--
+        MARK: vlp16-lidar
     -->
     <xacro:macro name="VLP-16" params="*origin parent">
@@ -97,5 +137,5 @@
                 <update_rate>10</update_rate>
                 <visualize>true</visualize>
-                <topic>velodyne_points</topic>
+                <topic>scan</topic>
                 <always_on>true</always_on>
                 <gz_frame_id>velodyne</gz_frame_id>

Commit message: figured out some localization stuff

File: src/igvc25/description/fwd.robot.xacro (robot description, xacro)
@@ -2,5 +2,6 @@
 <robot xmlns:xacro="http://www.ros.org/wiki/xacro" name="robot">
     <!-- Reusable properties -->
-    <xacro:property name="footprint_offset" value="0 0 -0.15875"/>
+    <!-- real offset = -0.15875, preted z0 = wheel height -->
+    <xacro:property name="footprint_offset" value="0 0 0"/>
     <xacro:property name="c_x"              value="0.9144"/>
     <xacro:property name="c_y"              value="0.6096"/>
