Commit message: ackemann paramaterization

File: src/igvc25/description/ackermann_linkage.urdf (robot description, URDF)
Before this commit: robot sarah7, 14 links, 13 joints
Links:
- link chassis_link: geometry visual box size=${chassis_length} ${chassis_width} ${chassis_height}
- link frame: geometry visual box size=${frame_length} ${frame_width} ${frame_thickness}
- link left_steering_arm: geometry visual box size=${steering_arm_width} ${steering_arm_length} ${steering_arm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
- link left_tie_rod: geometry visual box size=${tie_rod_width} ${tie_rod_length} ${tie_rod_thickness}
- link lf_wheel: geometry visual cylinder length=${wheel_length} radius=${wheel_radius}
- link lr_wheel: geometry visual cylinder length=${wheel_length} radius=${wheel_radius}
- link pinion: geometry visual cylinder length=${pinion_length} radius=${pinion_radius}
- link rack: geometry visual box size=${rack_width} ${rack_length} ${rack_thickness}
- link rf_wheel: geometry visual cylinder length=${wheel_length} radius=${wheel_radius}
- link right_steering_arm: geometry visual box size=${steering_arm_width} ${steering_arm_length} ${steering_arm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
- link right_tie_rod: geometry visual box size=${tie_rod_width} ${tie_rod_length} ${tie_rod_thickness}
- link rr_wheel: geometry visual cylinder length=${wheel_length} radius=${wheel_radius}
Joints:
- joint chassis_joint: origin xyz=-0.4572 0.0 0.0762 -> xyz=${chassis_offset_x} 0.0 ${chassis_offset_z}
- joint diff_j: origin xyz=-0.9144 0.0 0.0 -> xyz=${diff_offset_x} 0.0 0.0
- joint lf_wjoint: origin xyz=0.1 0.0 0.0 rpy=0.0 -1.57 0.0 -> xyz=${wheel_offset_x} 0.0 0.0 rpy=0.0 -1.57 0.0
- joint lr_wjoint: origin xyz=0.0 0.4048 0.0 rpy=-1.57 0.0 0.0 -> xyz=0.0 ${rear_wheel_spacing} 0.0 rpy=-1.57 0.0 0.0
- joint pin_four: origin xyz=0.0 -0.3045 0.0 -> xyz=0.0 ${pin_four_y} 0.0
- joint pin_one: origin xyz=0.0 0.3045 0.0 -> xyz=0.0 ${pin_one_y} 0.0
- joint pin_three: origin xyz=0.0 -0.1737 0.0 -> xyz=0.0 ${pin_three_y} 0.0
- joint pin_two: origin xyz=0.0 0.1737 0.0 -> xyz=0.0 ${pin_two_y} 0.0
- joint pinion_joint: limit lower=-1.586 upper=1.586 effort=0.0 velocity=0.0 -> lower=-${pinion_angle_limit} upper=${pinion_angle_limit} effort=0.0 velocity=0.0; origin xyz=-0.0315 0.0 0.04445 rpy=0.0 ${pi/2} 0.0 -> xyz=${pinion_offset_x} 0.0 ${pinion_offset_z} rpy=0.0 ${pi/2} 0.0
- joint rack_joint: limit lower=-0.03021 upper=0.03021 effort=0.0 velocity=0.0 -> lower=-${rack_travel_limit} upper=${rack_travel_limit} effort=0.0 velocity=0.0; origin xyz=-0.0315 0.0 0.0 -> xyz=${rack_offset_x} 0.0 0.0
- joint rf_wjoint: origin xyz=0.1 0.0 0.0 rpy=0.0 -1.57 0.0 -> xyz=${wheel_offset_x} 0.0 0.0 rpy=0.0 -1.57 0.0
- joint rr_wjoint: origin xyz=0.0 -0.4048 0.0 rpy=-1.57 0.0 0.0 -> xyz=0.0 -${rear_wheel_spacing} 0.0 rpy=-1.57 0.0 0.0

Commit message: new ackermann params

File: src/igvc25/description/ackermann_linkage.urdf (robot description, URDF)
Before this commit: robot sarah7, 14 links, 13 joints
Joints:
- joint lf_wjoint: origin xyz=${wheel_offset_x} 0.0 0.0 rpy=0.0 -1.57 0.0 -> xyz=${wheel_offset_x} 0.0 0.0 rpy=0.0 -1.57 -${wheel_angle}
- joint rf_wjoint: origin xyz=${wheel_offset_x} 0.0 0.0 rpy=0.0 -1.57 0.0 -> xyz=${wheel_offset_x} 0.0 0.0 rpy=0.0 -1.57 ${wheel_angle}

File: src/igvc25/description/macros/materials.xacro (robot description, xacro)
@@ -2,5 +2,5 @@
 <robot xmlns:xacro="http://www.ros.org/wiki/xacro">
     <material name="white">
-        <color rgba="1 1 1 1" />
+        <color rgba="1 1 1 0.1" />
     </material>
     <material name="black">
