Commit message: root test working
now need to add sensors + create different paths + catch in ros bags

File: src/igvc23/description/fwd.robot.xacro (robot description, xacro)
@@ -1,52 +1,52 @@
 <?xml version="1.0"?>
 <robot xmlns:xacro="http://www.ros.org/wiki/xacro" name="robot">
-    <!-- Reusable properties -->
-    <!-- real offset = -0.15875, preted z0 = wheel height -->
-    <xacro:property name="footprint_offset" value="0 0 0"/>
-    <xacro:property name="c_x"              value="0.9144"/>
-    <xacro:property name="c_y"              value="0.6096"/>
-    <xacro:property name="c_z"              value="0.1524"/>
-    <xacro:property name="chassis_size"     value="${c_x} ${c_y} ${c_z}"/>
-    <xacro:property name="chassis_mass"     value="13.6"/>
-    <xacro:property name="chassis_offset"   value="-0.2794 0 0.13688"/>
-    <xacro:property name="wheel_radius"     value="0.15875"/>
-    <xacro:property name="wheel_length"     value="0.06985"/>
-    <xacro:property name="wheel_mass"       value="1.0"/>
-    <xacro:property name="wheel_distance"   value="0.349725"/>
-    <xacro:property name="caster_radius"    value="0.15875"/>
-    <xacro:property name="caster_mass"      value="2.0"/>
-    <xacro:property name="caster_offset"    value="-0.57275349 0 0"/>
-    <joint name="footprint_joint" type="fixed">
-        <parent link="base_link"/>
-        <child link="base_footprint"/>
-        <origin xyz="${footprint_offset}"/>
-    </joint>
-    <!--
+  <!-- Reusable properties -->
+  <!-- real offset = -0.15875, preted z0 = wheel height -->
+  <xacro:property name="footprint_offset" value="0 0 0" />
+  <xacro:property name="c_x" value="0.9144" />
+  <xacro:property name="c_y" value="0.6096" />
+  <xacro:property name="c_z" value="0.1524" />
+  <xacro:property name="chassis_size" value="${c_x} ${c_y} ${c_z}" />
+  <xacro:property name="chassis_mass" value="13.6" />
+  <xacro:property name="chassis_offset" value="-0.2794 0 0.13688" />
+  <xacro:property name="wheel_radius" value="0.15875" />
+  <xacro:property name="wheel_length" value="0.06985" />
+  <xacro:property name="wheel_mass" value="1.0" />
+  <xacro:property name="wheel_distance" value="0.349725" />
+  <xacro:property name="caster_radius" value="0.15875" />
+  <xacro:property name="caster_mass" value="2.0" />
+  <xacro:property name="caster_offset" value="-0.57275349 0 0" />
+  <joint name="footprint_joint" type="fixed">
+    <parent link="base_link" />
+    <child link="base_footprint" />
+    <origin xyz="${footprint_offset}" />
+  </joint>
+  <!--
         MARK: Core
     -->
-    <!-- CHASSIS -->
-    <joint name="chassis_joint" type="fixed">
-        <parent link="base_link"/>
-        <child link="chassis_link"/>
-        <origin xyz="${chassis_offset}"/>
-    </joint>
-    <link name="chassis_link">
-        <xacro:inertial_box mass="${chassis_mass}" x="${c_x}" y="${c_y}" z="${c_z}">
-            <origin xyz="0 0 0" rpy="0 0 0" />
-        </xacro:inertial_box>
-        <visual>
-            <geometry>
-                <box size="${chassis_size}"/>
-            </geometry>
-            <material name="white"/>
-        </visual>
-        <collision>
-            <geometry>
-                <box size="${chassis_size}"/>
-            </geometry>
-        </collision>
-    </link>
-    <!-- DRIVE WHEELS -->
-    <xacro:wheel
+  <!-- CHASSIS -->
+  <joint name="chassis_joint" type="fixed">
+    <parent link="base_link" />
+    <child link="chassis_link" />
+    <origin xyz="${chassis_offset}" />
+  </joint>
+  <link name="chassis_link">
+    <xacro:inertial_box mass="${chassis_mass}" x="${c_x}" y="${c_y}" z="${c_z}">
+      <origin xyz="0 0 0" rpy="0 0 0" />
+    </xacro:inertial_box>
+    <visual>
+      <geometry>
+        <box size="${chassis_size}" />
+      </geometry>
+      <material name="white" />
+    </visual>
+    <collision>
+      <geometry>
+        <box size="${chassis_size}" />
+      </geometry>
+    </collision>
+  </link>
+  <!-- DRIVE WHEELS -->
+  <xacro:wheel
     name="left_wheel"
     parent_link="base_link"
@@ -54,6 +54,6 @@
     wheel_radius="${wheel_radius}"
     wheel_length="${wheel_length}"
-    wheel_mass="${wheel_mass}"/>
-    <xacro:wheel
+    wheel_mass="${wheel_mass}" />
+  <xacro:wheel
     name="right_wheel"
     parent_link="base_link"
@@ -61,128 +61,129 @@
     wheel_radius="${wheel_radius}"
     wheel_length="${wheel_length}"
-    wheel_mass="${wheel_mass}"/>
-    <!-- CASTER WHEEL -->
-    <joint name="caster_joint" type="fixed">
-        <parent link="base_link"/>
-        <child link="caster_link"/>
-        <origin xyz="${caster_offset}"/>
-    </joint>
-    <link name="caster_link">
-        <xacro:inertial_sphere mass="${caster_mass}" radius="${caster_radius}">
-            <origin xyz="0 0 0" rpy="0 0 0" />
-        </xacro:inertial_sphere>
-        <visual>
-            <geometry>
-                <sphere radius="${caster_radius}"/>
-            </geometry>
-            <material name="blue" />
-        </visual>
-        <collision>
-            <geometry>
-                <sphere radius="${caster_radius}"/>
-            </geometry>
-        </collision>
-    </link>
-    <!--
+    wheel_mass="${wheel_mass}" />
+  <!-- CASTER WHEEL -->
+  <joint name="caster_joint" type="fixed">
+    <parent link="base_link" />
+    <child link="caster_link" />
+    <origin xyz="${caster_offset}" />
+  </joint>
+  <link name="caster_link">
+    <xacro:inertial_sphere mass="${caster_mass}" radius="${caster_radius}">
+      <origin xyz="0 0 0" rpy="0 0 0" />
+    </xacro:inertial_sphere>
+    <visual>
+      <geometry>
+        <sphere radius="${caster_radius}" />
+      </geometry>
+      <material name="blue" />
+    </visual>
+    <collision>
+      <geometry>
+        <sphere radius="${caster_radius}" />
+      </geometry>
+    </collision>
+  </link>
+  <!--
         MARK: Sensors
     -->
-    <!-- Lidar -->
-    <xacro:lidar parent="base_link">
-        <origin xyz="-0.3 0 0.3" rpy="0 0 0"/>
-    </xacro:lidar>
-    <!-- IMU -->
-    <xacro:ph-imu parent="lidar_frame">
-        <origin xyz="0 0 0.05" rpy="0 0 0"/>
-    </xacro:ph-imu>
-    <!-- GPS -->
-    <xacro:garmin-gps parent="imu">
-        <origin xyz="0 0 0.05" rpy="0 0 0"/>
-    </xacro:garmin-gps>
-    <!-- Camera -->
-    <xacro:logi-cam parent="chassis_link" name="left_camera">
-        <origin xyz="0.5 ${wheel_distance} 0.05" rpy="0.0 0.0 0.523599"/>
-    </xacro:logi-cam>
-    <xacro:logi-cam parent="chassis_link" name="right_camera">
-        <origin xyz="0.5 -${wheel_distance} 0.05" rpy="0.0 0.0 -0.523599"/>
-    </xacro:logi-cam>
-    <!--
+  <!-- Lidar -->
+  <xacro:lidar parent="base_link">
+    <origin xyz="-0.3 0 0.3" rpy="0 0 0" />
+  </xacro:lidar>
+  <!-- IMU -->
+  <xacro:ph-imu parent="lidar_frame">
+    <origin xyz="0 0 0.05" rpy="0 0 0" />
+  </xacro:ph-imu>
+  <!-- GPS -->
+  <xacro:garmin-gps parent="imu">
+    <origin xyz="0 0 0.05" rpy="0 0 0" />
+  </xacro:garmin-gps>
+  <!-- Camera -->
+  <xacro:logi-cam parent="chassis_link" name="left_camera">
+    <origin xyz="0.5 ${wheel_distance} 0.05" rpy="0.0 0.0 0.523599" />
+  </xacro:logi-cam>
+  <xacro:logi-cam parent="chassis_link" name="right_camera">
+    <origin xyz="0.5 -${wheel_distance} 0.05" rpy="0.0 0.0 -0.523599" />
+  </xacro:logi-cam>
+  <!--
         MARK: Control
     -->
-    <xacro:unless value="$(arg simulation)">
-        <ros2_control name="RealRobot" type="system">
-            <hardware>
-                <plugin>diffdrive_arduino/DiffDriveArduinoHardware</plugin>
-                <param name="left_wheel_name">left_wheel_joint</param>
-                <param name="right_wheel_name">right_wheel_joint</param>
-                <param name="loop_rate">30</param>
-                <param name="device">/dev/ttyUSB0</param>
-                <param name="baud_rate">57600</param>
-                <param name="timeout_ms">1000</param>
-                <param name="enc_counts_per_rev">3436</param>
-            </hardware>
-            <joint name="left_wheel_joint">
-                <command_interface name="velocity">
-                    <param name="min">-10</param>
-                    <param name="max">10</param>
-                </command_interface>
-                <state_interface name="position"/>
-                <state_interface name="velocity"/>
-            </joint>
-            <joint name="right_wheel_joint">
-                <command_interface name="velocity">
-                    <param name="min">-10</param>
-                    <param name="max">10</param>
-                </command_interface>
-                <state_interface name="position"/>
-                <state_interface name="velocity"/>
-            </joint>
-        </ros2_control>
-    </xacro:unless>
-    <xacro:if value="$(arg simulation)">
-        <ros2_control name="GazeboSystem" type="system">
-            <hardware>
-                <plugin>gz_ros2_control/GazeboSimSystem</plugin>
-            </hardware>
-            <joint name="left_wheel_joint">
-                <command_interface name="velocity">
-                    <param name="min">-10</param>
-                    <param name="max">10</param>
-                </command_interface>
-                <state_interface name="velocity"/>
-                <state_interface name="position"/>
-            </joint>
-            <joint name="right_wheel_joint">
-                <command_interface name="velocity">
-                    <param name="min">-10</param>
-                    <param name="max">10</param>
-                </command_interface>
-                <state_interface name="velocity"/>
-                <state_interface name="position"/>
-            </joint>
-        </ros2_control>
-    </xacro:if>
-    <gazebo>
-        <plugin name="gz_ros2_control::GazeboSimROS2ControlPlugin" filename="libgz_ros2_control-system.so">
-            <parameters>$(find igvc23)/config/controllers.yaml</parameters>
-            <parameters>$(find igvc23)/config/controllers_sim.yaml</parameters>
-        </plugin>
-    </gazebo>
-    <!--
+  <xacro:unless value="$(arg simulation)">
+    <ros2_control name="RealRobot" type="system">
+      <hardware>
+        <plugin>diffdrive_arduino/DiffDriveArduinoHardware</plugin>
+        <param name="left_wheel_name">left_wheel_joint</param>
+        <param name="right_wheel_name">right_wheel_joint</param>
+        <param name="loop_rate">30</param>
+        <param name="device">/dev/ttyUSB0</param>
+        <param name="baud_rate">57600</param>
+        <param name="timeout_ms">1000</param>
+        <param name="enc_counts_per_rev">3436</param>
+      </hardware>
+      <joint name="left_wheel_joint">
+        <command_interface name="velocity">
+          <param name="min">-10</param>
+          <param name="max">10</param>
+        </command_interface>
+        <state_interface name="position" />
+        <state_interface name="velocity" />
+      </joint>
+      <joint name="right_wheel_joint">
+        <command_interface name="velocity">
+          <param name="min">-10</param>
+          <param name="max">10</param>
+        </command_interface>
+        <state_interface name="position" />
+        <state_interface name="velocity" />
+      </joint>
+    </ros2_control>
+  </xacro:unless>
+  <xacro:if value="$(arg simulation)">
+    <ros2_control name="GazeboSystem" type="system">
+      <hardware>
+        <plugin>gz_ros2_control/GazeboSimSystem</plugin>
+      </hardware>
+      <joint name="left_wheel_joint">
+        <command_interface name="velocity">
+          <param name="min">-10</param>
+          <param name="max">10</param>
+        </command_interface>
+        <state_interface name="velocity" />
+        <state_interface name="position" />
+      </joint>
+      <joint name="right_wheel_joint">
+        <command_interface name="velocity">
+          <param name="min">-10</param>
+          <param name="max">10</param>
+        </command_interface>
+        <state_interface name="velocity" />
+        <state_interface name="position" />
+      </joint>
+    </ros2_control>
+  </xacro:if>
+  <gazebo>
+    <plugin name="gz_ros2_control::GazeboSimROS2ControlPlugin"
+      filename="libgz_ros2_control-system.so">
+      <parameters>$(find igvc23)/config/controllers.yaml</parameters>
+      <parameters>$(find igvc23)/config/controllers_sim.yaml</parameters>
+    </plugin>
+  </gazebo>
+  <!--
         MARK: Sim
     -->
-    <!-- Simulation References -->
-    <gazebo reference="chassis_link">
-        <material>Gazebo/White</material>
-    </gazebo>
-    <gazebo reference="left_wheel">
-        <material>Gazebo/Blue</material>
-    </gazebo>
-    <gazebo reference="right_wheel">
-        <material>Gazebo/Blue</material>
-    </gazebo>
-    <gazebo reference="caster_link">
-        <material>Gazebo/Blue</material>
-        <mu1 value="0.001"/>
-        <mu2 value="0.001"/>
-    </gazebo>
+  <!-- Simulation References -->
+  <gazebo reference="chassis_link">
+    <material>Gazebo/White</material>
+  </gazebo>
+  <gazebo reference="left_wheel">
+    <material>Gazebo/Blue</material>
+  </gazebo>
+  <gazebo reference="right_wheel">
+    <material>Gazebo/Blue</material>
+  </gazebo>
+  <gazebo reference="caster_link">
+    <material>Gazebo/Blue</material>
+    <mu1 value="0.001" />
+    <mu2 value="0.001" />
+  </gazebo>
 </robot>
