Commit message: tests might work

File: src/igvc25/description/macros/components.xacro (robot description, xacro)
@@ -1,123 +1,125 @@
 <?xml version="1.0"?>
-<robot xmlns:xacro="http://www.ros.org/wiki/xacro" >
-    <!--
+<robot xmlns:xacro="http://www.ros.org/wiki/xacro">
+  <!--
         MARK: wheel
     -->
-    <xacro:macro name="wheel" params="name parent_link wheel_distance wheel_radius wheel_length wheel_mass">
-        <joint name="${name}_joint" type="continuous">
-            <parent link="${parent_link}"/>
-            <child link="${name}"/>
-            <origin xyz="0 ${wheel_distance} 0" rpy="-${pi/2} 0 0"/>
-            <axis xyz="0 0 1"/>
-        </joint>
-        <link name="${name}">
-            <xacro:inertial_cylinder mass="${wheel_mass}" radius="${wheel_radius}" length="${wheel_length}">
-                <origin xyz="0 0 0" rpy="0 0 0" />
-            </xacro:inertial_cylinder>
-            <visual>
-                <geometry>
-                    <cylinder radius="${wheel_radius}" length="${wheel_length}"/>
-                </geometry>
-                <material name="blue"/>
-            </visual>
-            <collision>
-                <geometry>
-                    <cylinder radius="${wheel_radius}" length="${wheel_length}"/>
-                </geometry>
-            </collision>
-        </link>
-    </xacro:macro>
-    <!--
+  <xacro:macro name="wheel"
+    params="name parent_link wheel_distance wheel_radius wheel_length wheel_mass">
+    <joint name="${name}_joint" type="continuous">
+      <parent link="${parent_link}" />
+      <child link="${name}" />
+      <origin xyz="0 ${wheel_distance} 0" rpy="-${pi/2} 0 0" />
+      <axis xyz="0 0 1" />
+    </joint>
+    <link name="${name}">
+      <xacro:inertial_cylinder mass="${wheel_mass}" radius="${wheel_radius}"
+        length="${wheel_length}">
+        <origin xyz="0 0 0" rpy="0 0 0" />
+      </xacro:inertial_cylinder>
+      <visual>
+        <geometry>
+          <cylinder radius="${wheel_radius}" length="${wheel_length}" />
+        </geometry>
+        <material name="blue" />
+      </visual>
+      <collision>
+        <geometry>
+          <cylinder radius="${wheel_radius}" length="${wheel_length}" />
+        </geometry>
+      </collision>
+    </link>
+  </xacro:macro>
+  <!--
         MARK: flat-lidar
     -->
-    <xacro:macro name="lidar" params="*origin parent">
-        <joint name="lidar_joint" type="fixed">
-            <parent link="${parent}"/>
-            <child link="lidar_frame"/>
-            <xacro:insert_block name="origin"/>
-        </joint>
-        <link name="lidar_frame">
-            <visual>
-                <geometry>
-                    <cylinder radius="0.05" length="0.04"/>
-                </geometry>
-                <material name="black"/>
-            </visual>
-        </link>
-        <gazebo reference="lidar_frame">
-            <sensor name="laser" type="gpu_lidar">
-                <pose> 0 0 0 0 0 0 </pose>
-                <visualize>false</visualize>
-                <update_rate>10</update_rate>
-                <lidar>
-                    <scan>
-                        <horizontal>
-                            <samples>360</samples>
-                            <min_angle>-3.14</min_angle>
-                            <max_angle>3.14</max_angle>
-                        </horizontal>
-                    </scan>
-                    <range>
-                        <min>0.3</min>
-                        <max>12</max>
-                    </range>
-                </lidar>
-                <topic>scan</topic>
-                <gz_frame_id>lidar_frame</gz_frame_id>
-            </sensor>
-        </gazebo>
-    </xacro:macro>
-    <!--
+  <xacro:macro name="lidar" params="*origin parent">
+    <joint name="lidar_joint" type="fixed">
+      <parent link="${parent}" />
+      <child link="lidar_frame" />
+      <xacro:insert_block name="origin" />
+    </joint>
+    <link name="lidar_frame">
+      <visual>
+        <geometry>
+          <cylinder radius="0.05" length="0.04" />
+        </geometry>
+        <material name="black" />
+      </visual>
+    </link>
+    <gazebo reference="lidar_frame">
+      <sensor name="laser" type="gpu_lidar">
+        <pose> 0 0 0 0 0 0 </pose>
+        <visualize>false</visualize>
+        <update_rate>10</update_rate>
+        <lidar>
+          <scan>
+            <horizontal>
+              <samples>360</samples>
+              <min_angle>-3.14</min_angle>
+              <max_angle>3.14</max_angle>
+            </horizontal>
+          </scan>
+          <range>
+            <min>0.3</min>
+            <max>12</max>
+          </range>
+        </lidar>
+        <topic>scan</topic>
+        <gz_frame_id>lidar_frame</gz_frame_id>
+      </sensor>
+    </gazebo>
+  </xacro:macro>
+  <!--
         MARK: vlp16-lidar
     -->
-    <xacro:macro name="VLP-16" params="*origin parent">
-        <!-- VLP-16 LiDAR -->
-        <!-- meshes seems to be broken, using simple geometry instead -->
-        <joint name="velodyne_base_mount_joint" type="fixed">
-            <xacro:insert_block name="origin" />
-            <parent link="${parent}"/>
-            <child link="velodyne_base_link"/>
-        </joint>
-        <link name="velodyne_base_link">
-            <inertial>
-                <mass value="0.83"/>
-                <origin xyz="0 0 0.03585"/>
-                <inertia ixx="${(0.83 * (3.0*0.0516*0.0516 + 0.0717*0.0717)) / 12.0}" ixy="0" ixz="0"
-                iyy="${(0.83 * (3.0*0.0516*0.0516 + 0.0717*0.0717)) / 12.0}" iyz="0"
-                izz="${0.5 * 0.83 * (0.0516*0.0516)}"/>
-            </inertial>
-            <visual>
-                <!-- <geometry>
+  <xacro:macro name="VLP-16" params="*origin parent">
+    <!-- VLP-16 LiDAR -->
+    <!-- meshes seems to be broken, using simple geometry instead -->
+    <joint name="velodyne_base_mount_joint" type="fixed">
+      <xacro:insert_block name="origin" />
+      <parent link="${parent}" />
+      <child link="velodyne_base_link" />
+    </joint>
+    <link name="velodyne_base_link">
+      <inertial>
+        <mass value="0.83" />
+        <origin xyz="0 0 0.03585" />
+        <inertia ixx="${(0.83 * (3.0*0.0516*0.0516 + 0.0717*0.0717)) / 12.0}" ixy="0" ixz="0"
+          iyy="${(0.83 * (3.0*0.0516*0.0516 + 0.0717*0.0717)) / 12.0}" iyz="0"
+          izz="${0.5 * 0.83 * (0.0516*0.0516)}" />
+      </inertial>
+      <visual>
+        <!-- <geometry>
                     <mesh filename="${mesh_folder}/VLP16_base_1.dae"/>
                 </geometry> -->
-                <geometry>
-                    <cylinder radius="${0.103 / 2.0}" length="0.072"/>
-                </geometry>
-                <material name="black"/>
-            </visual>
-            <!-- <visual>
+        <geometry>
+          <cylinder radius="${0.103 / 2.0}" length="0.072" />
+        </geometry>
+        <material name="black" />
+      </visual>
+      <!-- <visual>
                 <geometry>
                     <mesh filename="${mesh_folder}/VLP16_base_2.dae"/>
                 </geometry>
             </visual> -->
-            <collision>
-                <origin rpy="0 0 0" xyz="0 0 0.03585"/>
-                <geometry>
-                    <cylinder radius="0.0516" length="0.0717"/>
-                </geometry>
-            </collision>
-        </link>
-        <joint name="velodyne_base_scan_joint" type="fixed" >
-            <origin xyz="0 0 0.0377" rpy="0 0 0" />
-            <parent link="velodyne_base_link" />
-            <child link="velodyne"/>
-        </joint>
-        <link name="velodyne">
-            <inertial>
-                <mass value="0.01"/>
-                <origin xyz="0 0 0"/>
-                <inertia ixx="1e-7" ixy="0" ixz="0" iyy="1e-7" iyz="0" izz="1e-7"/>
-            </inertial>
-            <!-- <visual>
+      <collision>
+        <origin rpy="0 0 0" xyz="0 0 0.03585" />
+        <geometry>
+          <cylinder radius="0.0516" length="0.0717" />
+        </geometry>
+      </collision>
+    </link>
+    <joint name="velodyne_base_scan_joint" type="fixed">
+      <origin xyz="0 0 0.0377" rpy="0 0 0" />
+      <parent link="velodyne_base_link" />
+      <child link="velodyne" />
+    </joint>
+    <link name="velodyne">
+      <inertial>
+        <mass value="0.01" />
+        <origin xyz="0 0 0" />
+        <inertia ixx="1e-7" ixy="0" ixz="0" iyy="1e-7" iyz="0" izz="1e-7" />
+      </inertial>
+      <!-- <visual>
                 <origin xyz="0 0 -0.0377"/>
                 <geometry>
@@ -125,160 +127,161 @@
                 </geometry>
             </visual> -->
-            <collision>
-                <geometry>
-                    <sphere radius="0"/>
-                </geometry>
-            </collision>
-        </link>
-        <!-- Gazebo requires ... -->
-        <gazebo reference="velodyne">
-            <sensor name="velodyne" type="gpu_lidar">
-                <pose>0 0 0 0 0 0</pose>
-                <update_rate>10</update_rate>
-                <visualize>true</visualize>
-                <topic>scan</topic>
-                <always_on>true</always_on>
-                <gz_frame_id>velodyne</gz_frame_id>
-                <ray>
-                    <scan>
-                        <horizontal>
-                            <samples>1800</samples>
-                            <resolution>1</resolution>
-                            <min_angle>-3.14159</min_angle>
-                            <max_angle>3.14159</max_angle>
-                        </horizontal>
-                        <vertical>
-                            <samples>16</samples>
-                            <resolution>1</resolution>
-                            <min_angle>-0.261799</min_angle> <!-- -15 degrees -->
-                            <max_angle>0.261799</max_angle>  <!-- +15 degrees -->
-                        </vertical>
-                    </scan>
-                    <range>
-                        <min>0.1</min>
-                        <max>100.0</max>
-                        <resolution>0.01</resolution>
-                    </range>
-                    <noise>
-                        <type>gaussian</type>
-                        <mean>0.0</mean>
-                        <stddev>0.01</stddev>
-                    </noise>
-                </ray>
-            </sensor>
-        </gazebo>
-    </xacro:macro>
-    <!--
+      <collision>
+        <geometry>
+          <sphere radius="0" />
+        </geometry>
+      </collision>
+    </link>
+    <!-- Gazebo requires ... -->
+    <gazebo reference="velodyne">
+      <sensor name="velodyne" type="gpu_lidar">
+        <pose>0 0 0 0 0 0</pose>
+        <update_rate>10</update_rate>
+        <visualize>true</visualize>
+        <topic>scan</topic>
+        <always_on>true</always_on>
+        <gz_frame_id>velodyne</gz_frame_id>
+        <ray>
+          <scan>
+            <horizontal>
+              <samples>1800</samples>
+              <resolution>1</resolution>
+              <min_angle>-3.14159</min_angle>
+              <max_angle>3.14159</max_angle>
+            </horizontal>
+            <vertical>
+              <samples>16</samples>
+              <resolution>1</resolution>
+              <min_angle>-0.261799</min_angle> <!-- -15 degrees -->
+              <max_angle>0.261799</max_angle>  <!-- +15 degrees -->
+            </vertical>
+          </scan>
+          <range>
+            <min>0.1</min>
+            <max>100.0</max>
+            <resolution>0.01</resolution>
+          </range>
+          <noise>
+            <type>gaussian</type>
+            <mean>0.0</mean>
+            <stddev>0.01</stddev>
+          </noise>
+        </ray>
+      </sensor>
+    </gazebo>
+  </xacro:macro>
+  <!--
         MARK: imu
     -->
-    <!-- https://www.phidgets.com/productfiles/MOT0110/MOT0110_0/Documentation/MOT0110_0_Mechanical.pdf -->
-    <xacro:macro name="ph-imu" params="*origin parent">
-        <joint name="imu_joint" type="fixed">
-            <parent link="${parent}"/>
-            <child link="imu"/>
-            <xacro:insert_block name="origin"/>
-        </joint>
-        <link name="imu">
-            <visual>
-                <geometry>
-                    <box size="0.038989 0.037846 0.013380"/>
-                </geometry>
-                <material name="orange"/>
-            </visual>
-        </link>
-        <gazebo reference="imu">
-            <sensor name="imu" type="imu">
-                <pose>0 0 0 0 0 0</pose>
-                <always_on>true</always_on>
-                <update_rate>1</update_rate>
-                <visualize>true</visualize>
-                <topic>imu</topic>
-                <gz_frame_id>imu</gz_frame_id>
-                <plugin
-                    filename="gz-sim-imu-system"
-                    name="gz::sim::systems::Imu">
-                </plugin>
-            </sensor>
-        </gazebo>
-    </xacro:macro>
-    <!--
+  <!--
+  https://www.phidgets.com/productfiles/MOT0110/MOT0110_0/Documentation/MOT0110_0_Mechanical.pdf -->
+  <xacro:macro name="ph-imu" params="*origin name parent">
+    <joint name="imu_joint" type="fixed">
+      <parent link="${parent}" />
+      <child link="${name}" />
+      <xacro:insert_block name="origin" />
+    </joint>
+    <link name="${name}">
+      <visual>
+        <geometry>
+          <box size="0.038989 0.037846 0.013380" />
+        </geometry>
+        <material name="orange" />
+      </visual>
+    </link>
+    <gazebo reference="${name}">
+      <sensor name="imu" type="imu">
+        <pose>0 0 0 0 0 0</pose>
+        <always_on>true</always_on>
+        <update_rate>1</update_rate>
+        <visualize>true</visualize>
+        <topic>imu</topic>
+        <gz_frame_id>imu</gz_frame_id>
+        <plugin
+          filename="gz-sim-imu-system"
+          name="gz::sim::systems::Imu">
+        </plugin>
+      </sensor>
+    </gazebo>
+  </xacro:macro>
+  <!--
         MARK: GPS
     -->
-    <!-- https://www.garmin.com/en-US/p/27594#overview -->
-    <xacro:macro name="garmin-gps" params="*origin parent">
-        <joint name="gps_joint" type="fixed">
-            <parent link="${parent}"/>
-            <child link="gps"/>
-            <xacro:insert_block name="origin"/>
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
Commit message: ackermann urdf

File: src/igvc25/description/macros/components.xacro (robot description, xacro)
@@ -5,12 +5,14 @@
     -->
   <xacro:macro name="wheel"
-    params="name parent_link wheel_distance wheel_radius wheel_length wheel_mass">
+    params="name parent_link wheel_distance wheel_radius wheel_length wheel_mass wheel_orientation max_effort max_vel">
     <joint name="${name}_joint" type="continuous">
       <parent link="${parent_link}" />
-      <child link="${name}" />
-      <origin xyz="0 ${wheel_distance} 0" rpy="-${pi/2} 0 0" />
+      <child link="${name}_link" />
+      <origin xyz="0 ${wheel_distance} 0" rpy="${wheel_orientation} 0 0" />
       <axis xyz="0 0 1" />
-    </joint>
-    <link name="${name}">
+      <limit effort="${max_effort}" velocity="${max_vel}"/>
+      <dynamics damping="0.1" friction="0.1"/>
+    </joint>
+    <link name="${name}_link">
       <xacro:inertial_cylinder mass="${wheel_mass}" radius="${wheel_radius}"
         length="${wheel_length}">
