Commit message: urdf 3.0 start

File: src/igvc/description/macros/components.xacro (robot description, xacro)
@@ -26,4 +26,34 @@
       </visual>
       <collision>
+        <geometry>
+          <cylinder radius="${wheel_radius}" length="${wheel_length}" />
+        </geometry>
+      </collision>
+    </link>
+  </xacro:macro>
+  <!--
+        MARK: steer
+    -->
+  <xacro:macro name="steer" params="*origin name parent_link wheel_radius wheel_length wheel_mass">
+    <joint name="${name}_steering_joint" type="revolute">
+      <parent link="${parent_link}"/>
+      <child link="${name}_link"/>
+      <xacro:insert_block name="origin" />
+      <axis xyz="0 0 1"/>
+    </joint>
+    <link name="${name}_wheel">
+      <xacro:inertial_cylinder mass="${wheel_mass}" radius="${wheel_radius}"
+        length="${wheel_length}">
+        <origin xyz="0 0 0" rpy="-${pi/2} 0 0" />
+      </xacro:inertial_cylinder>
+      <visual>
+        <origin xyz="0 0 0" rpy="-${pi/2} 0 0" />
+        <geometry>
+          <cylinder radius="${wheel_radius}" length="${wheel_length}" />
+        </geometry>
+        <material name="blue" />
+      </visual>
+      <collision>
+        <origin xyz="0 0 0" rpy="-${pi/2} 0 0" />
         <geometry>
           <cylinder radius="${wheel_radius}" length="${wheel_length}" />

Commit message: encoder dix??

File: src/igvc/description/macros/components.xacro (robot description, xacro)
@@ -200,41 +200,4 @@
       </collision>
     </link>
-    <!-- Gazebo requires ... -->
-    <!-- <gazebo reference="velodyne">
-      <sensor name="velodyne" type="gpu_lidar">
-        <pose>0 0 0 0 0 0</pose>
-        <update_rate>10</update_rate>
-        <visualize>true</visualize>
-        <topic>scan</topic>
-        <always_on>true</always_on>
-        <gz_frame_id>velodyne</gz_frame_id>
-        <ray>
-          <scan>
-            <horizontal>
-              <samples>1800</samples>
-              <resolution>1</resolution>
-              <min_angle>-3.14159</min_angle>
-              <max_angle>3.14159</max_angle>
-            </horizontal>
-            <vertical>
-              <samples>16</samples>
-              <resolution>1</resolution>
-              <min_angle>-0.261799</min_angle> <!-- -15 degrees -->
-              <max_angle>0.261799</max_angle>  <!-- +15 degrees -->
-            </vertical>
-          </scan>
-          <range>
-            <min>0.1</min>
-            <max>100.0</max>
-            <resolution>0.01</resolution>
-          </range>
-          <noise>
-            <type>gaussian</type>
-            <mean>0.0</mean>
-            <stddev>0.01</stddev>
-          </noise>
-        </ray>
-      </sensor>
-    </gazebo> -->
   </xacro:macro>
   <!--
@@ -244,5 +207,5 @@
   https://www.phidgets.com/productfiles/MOT0110/MOT0110_0/Documentation/MOT0110_0_Mechanical.pdf -->
   <xacro:macro name="ph-imu" params="*origin name parent">
-    <joint name="imu_joint" type="fixed">
+    <joint name="${name}_joint" type="fixed">
       <parent link="${parent}" />
       <child link="${name}" />
@@ -257,5 +220,5 @@
       </visual>
     </link>
-    <gazebo reference="${name}">
+    <!-- <gazebo reference="${name}">
       <sensor name="imu" type="imu">
         <pose>0 0 0 0 0 0</pose>
@@ -269,5 +232,5 @@
         </plugin>
       </sensor>
-    </gazebo>
+    </gazebo> -->
   </xacro:macro>
   <!--
@@ -289,14 +252,13 @@
       </visual>
     </link>
-    <gazebo reference="gps">
+    <!-- <gazebo reference="gps">
       <sensor name="gps" type="navsat">
         <pose>0 0 0 0 0 0</pose>
         <always_on>true</always_on>
         <update_rate>1</update_rate>
-        <!-- <visualize>true</visualize> -->
         <topic>gps</topic>
         <gz_frame_id>gps</gz_frame_id>
       </sensor>
-    </gazebo>
+    </gazebo> -->
   </xacro:macro>
   <!--
