Commit message: new urdf

File: src/igvc/description/ackermann_ac.urdf (robot description, URDF)
Before this commit: robot igvc25, 1 links, 0 joints
Links:
- added link diff_link
- added link motor; visual cylinder length=0.025 radius=0.05
- added link pinion; visual cylinder length=0.025 radius=0.05
Joints:
- added joint diff_joint: type fixed, parent base_link, child diff_link, origin xyz=-${track_width} 0 0
- added joint motor_joint: type continuous, parent diff_link, child motor, origin xyz=0.0 0.0 0.1 rpy=0.0 -${pi/2} 0.0, axis 0 0 1
- added joint pinion_joint: type continuous, parent base_link, child pinion, origin xyz=0.0 0.0 0.1 rpy=0.0 -${pi/2} 0.0, axis 0 0 1

File: src/igvc/description/macros/components.xacro (robot description, xacro)
@@ -11,6 +11,6 @@
       <origin xyz="0 ${wheel_distance} 0" rpy="${wheel_orientation} 0 0" />
       <axis xyz="0 0 1" />
-      <limit effort="${max_effort}" velocity="${max_vel}"/>
-      <dynamics damping="0.1" friction="0.1"/>
+      <limit effort="${max_effort}" velocity="${max_vel}" />
+      <dynamics damping="0.1" friction="0.1" />
     </joint>
     <link name="${name}_link">
@@ -32,21 +32,18 @@
     </link>
   </xacro:macro>
-  <!--
-        MARK: steer
-    -->
-  <xacro:macro name="steer" params="*origin name parent_link wheel_radius wheel_length wheel_mass">
-    <joint name="${name}_steering_joint" type="revolute">
-      <parent link="${parent_link}"/>
-      <child link="${name}_link"/>
-      <xacro:insert_block name="origin" />
-      <axis xyz="0 0 1"/>
+  <xacro:macro name="wheel2"
+    params="name parent_link wheel_offset wheel_radius wheel_length wheel_mass">
+    <joint name="${name}_wheel_joint" type="continuous">
+      <parent link="${parent_link}" />
+      <child link="${name}_wheel" />
+      <origin xyz="0 ${wheel_offset} 0" rpy="-${pi/2} 0 0" />
+      <axis xyz="0 0 1" />
     </joint>
     <link name="${name}_wheel">
       <xacro:inertial_cylinder mass="${wheel_mass}" radius="${wheel_radius}"
         length="${wheel_length}">
-        <origin xyz="0 0 0" rpy="-${pi/2} 0 0" />
+        <origin xyz="0 0 0" rpy="0 0 0" />
       </xacro:inertial_cylinder>
       <visual>
-        <origin xyz="0 0 0" rpy="-${pi/2} 0 0" />
         <geometry>
           <cylinder radius="${wheel_radius}" length="${wheel_length}" />
@@ -55,5 +52,43 @@
       </visual>
       <collision>
-        <origin xyz="0 0 0" rpy="-${pi/2} 0 0" />
+        <geometry>
+          <cylinder radius="${wheel_radius}" length="${wheel_length}" />
+        </geometry>
+      </collision>
+    </link>
+  </xacro:macro>
+  <!--
+        MARK: steer
+    -->
+  <xacro:macro name="steer"
+    params="*origin name parent_link wheel_radius wheel_length wheel_mass wheel_offset">
+    <joint name="${name}_steering_joint" type="continuous">
+      <parent link="${parent_link}" />
+      <child link="${name}_steering_knuckle" />
+      <xacro:insert_block name="origin" />
+      <axis xyz="0 0 1" />
+    </joint>
+    <link name="${name}_steering_knuckle">
+      <!-- <xacro:inertial_box mass="0.1" x="0.01" y="0.01" z="0.1">
+        <origin xyz="0 0 0" />
+      </xacro:inertial_box> -->
+    </link>
+    <joint name="${name}_wheel_mount" type="fixed">
+      <parent link="${name}_steering_knuckle" />
+      <child link="${name}_wheel" />
+      <origin xyz="0 ${wheel_offset} 0" rpy="-${pi/2} 0 0" />
+    </joint>
+    <link name="${name}_wheel">
+      <xacro:inertial_cylinder mass="${wheel_mass}" radius="${wheel_radius}"
+        length="${wheel_length}">
+        <origin xyz="0 0 0" />
+      </xacro:inertial_cylinder>
+      <visual>
+        <geometry>
+          <cylinder radius="${wheel_radius}" length="${wheel_length}" />
+        </geometry>
+        <material name="blue" />
+      </visual>
+      <collision>
         <geometry>
           <cylinder radius="${wheel_radius}" length="${wheel_length}" />

Commit message: ctrl launch file

File: src/igvc/description/ackermann_ac.urdf (robot description, URDF)
Before this commit: robot igvc25, 4 links, 3 joints
Joints:
- removed joint motor_joint
- added joint rear_motor_joint: type continuous, parent diff_link, child motor, origin xyz=0.0 0.0 0.1 rpy=0.0 -${pi/2} 0.0, axis 0 0 1

Commit message: cleanup igvc control

File: src/igvc/description/ackermann_ac.urdf (robot description, URDF)
Before this commit: robot igvc25, 4 links, 3 joints
Joints:
- removed joint rear_motor_joint
- added joint motor_joint: type continuous, parent diff_link, child motor, origin xyz=0.0 0.0 0.1 rpy=0.0 -${pi/2} 0.0, axis 0 0 1

Commit message: cleanup vision launch and some configs

File: src/igvc/description/ackermann_ac.urdf (robot description, URDF)
Before this commit: robot igvc25, 4 links, 3 joints
Links:
- added link base_footprint
- added link chassis
Joints:
- added joint chassis_joint: type fixed, parent base_link, child chassis, origin xyz=-0.4575 0.0, 0.1955 rpy=0.0 -0.0208 0.0
- added joint footprint_joint: type None, parent base_link, child base_footprint, origin xyz=0.0 0.0 -0.1014 rpy=0.0 0.0 0.0
- joint diff_joint: origin xyz=-${track_width} 0 0 -> xyz=-0.815 0 0
- joint motor_joint: origin xyz=0.0 0.0 0.1 rpy=0.0 -${pi/2} 0.0 -> xyz=0.0 0.0 0.1955 rpy=0.0 -${pi/2} 0.0
- joint pinion_joint: origin xyz=0.0 0.0 0.1 rpy=0.0 -${pi/2} 0.0 -> xyz=0.0 0.0 0.1955 rpy=0.0 -${pi/2} 0.0

Commit message: restore gz sim

File: src/igvc/description/ackermann_ac.urdf (robot description, URDF)
Before this commit: robot igvc25, 6 links, 5 joints
Joints:
- joint chassis_joint: origin xyz=-0.4575 0.0, 0.1955 rpy=0.0 -0.0208 0.0 -> xyz=-0.4575 0.0 0.1955 rpy=0.0 -0.0208 0.0

File: src/igvc/description/macros/components.xacro (robot description, xacro)
@@ -100,5 +100,6 @@
         MARK: flat-lidar
     -->
-  <xacro:macro name="lidar" params="*origin parent">
+  <!-- Planar 2D lidar for Gazebo Sim → ros_gz_bridge → sensor_msgs/LaserScan on ${topic} -->
+  <xacro:macro name="lidar" params="*origin parent topic:=scan samples:=720">
     <joint name="lidar_joint" type="fixed">
       <parent link="${parent}" />
@@ -115,23 +116,31 @@
     </link>
     <gazebo reference="lidar_frame">
-      <sensor name="laser" type="gpu_lidar">
-        <pose> 0 0 0 0 0 0 </pose>
+      <sensor name="planar_lidar" type="gpu_lidar">
+        <pose>0 0 0 0 0 0</pose>
+        <topic>${topic}</topic>
+        <update_rate>20</update_rate>
+        <gz_frame_id>lidar_frame</gz_frame_id>
         <visualize>false</visualize>
-        <update_rate>10</update_rate>
-        <ray>
+        <always_on>true</always_on>
+        <lidar>
           <scan>
             <horizontal>
-              <samples>360</samples>
-              <min_angle>-3.14</min_angle>
-              <max_angle>3.14</max_angle>
+              <samples>${samples}</samples>
+              <resolution>1</resolution>
+              <min_angle>-3.14159265</min_angle>
+              <max_angle>3.14159265</max_angle>
             </horizontal>
+            <vertical>
+              <samples>1</samples>
+              <resolution>0.01</resolution>
+              <min_angle>0</min_angle>
+              <max_angle>0</max_angle>
+            </vertical>
           </scan>
           <range>
-            <min>0.3</min>
-            <max>12</max>
+            <min>0.12</min>
+            <max>30.0</max>
           </range>
-        </ray>
-        <topic>scan</topic>
-        <gz_frame_id>lidar_frame</gz_frame_id>
+        </lidar>
       </sensor>
     </gazebo>
@@ -140,13 +149,13 @@
         MARK: vlp16-lidar
     -->
-  <xacro:macro name="VLP-16" params="*origin parent">
+  <xacro:macro name="VLP-16" params="*origin parent name_prefix:='' lidar_topic:='velodyne_scan'">
     <!-- VLP-16 LiDAR -->
     <!-- meshes seems to be broken, using simple geometry instead -->
-    <joint name="velodyne_base_mount_joint" type="fixed">
-      <xacro:insert_block name="origin" />
-      <parent link="${parent}" />
-      <child link="velodyne_base_link" />
-    </joint>
-    <link name="velodyne_base_link">
+    <joint name="${name_prefix}velodyne_base_mount_joint" type="fixed">
+      <xacro:insert_block name="origin" />
+      <parent link="${parent}" />
+      <child link="${name_prefix}velodyne_base_link" />
+    </joint>
+    <link name="${name_prefix}velodyne_base_link">
       <inertial>
         <mass value="0.83" />
@@ -177,10 +186,10 @@
       </collision>
     </link>
-    <joint name="velodyne_base_scan_joint" type="fixed">
+    <joint name="${name_prefix}velodyne_base_scan_joint" type="fixed">
       <origin xyz="0 0 0.0377" rpy="0 0 0" />
-      <parent link="velodyne_base_link" />
-      <child link="velodyne" />
-    </joint>
-    <link name="velodyne">
+      <parent link="${name_prefix}velodyne_base_link" />
+      <child link="${name_prefix}velodyne" />
+    </joint>
+    <link name="${name_prefix}velodyne">
       <inertial>
         <mass value="0.01" />
@@ -200,4 +209,35 @@
       </collision>
     </link>
+    <!-- Gazebo Sim: planar spinning lidar (PoC obstacle detection / LaserScan bridge) -->
+    <gazebo reference="${name_prefix}velodyne">
+      <sensor name="${name_prefix}vlp16_gpu_lidar" type="gpu_lidar">
+        <pose>0 0 0 0 0 0</pose>
+        <update_rate>15</update_rate>
+        <topic>${lidar_topic}</topic>
+        <gz_frame_id>${name_prefix}velodyne</gz_frame_id>
+        <always_on>true</always_on>
+        <visualize>false</visualize>
+        <lidar>
+          <scan>
+            <horizontal>
+              <samples>720</samples>
+              <resolution>1</resolution>
+              <min_angle>-3.14159265</min_angle>
+              <max_angle>3.14159265</max_angle>
+            </horizontal>
+            <vertical>
+              <samples>1</samples>
+              <resolution>0.01</resolution>
+              <min_angle>0</min_angle>
+              <max_angle>0</max_angle>
+            </vertical>
+          </scan>
+          <range>
+            <min>0.2</min>
+            <max>50.0</max>
+          </range>
+        </lidar>
+      </sensor>
+    </gazebo>
   </xacro:macro>
   <!--
@@ -238,11 +278,11 @@
     -->
   <!-- https://www.garmin.com/en-US/p/27594#overview -->
-  <xacro:macro name="garmin-gps" params="*origin parent">
-    <joint name="gps_joint" type="fixed">
-      <parent link="${parent}" />
-      <child link="gps" />
-      <xacro:insert_block name="origin" />
-    </joint>
-    <link name="gps">
+  <xacro:macro name="garmin-gps" params="*origin parent name_prefix:=''">
+    <joint name="${name_prefix}gps_joint" type="fixed">
+      <parent link="${parent}" />
+      <child link="${name_prefix}gps" />
+      <xacro:insert_block name="origin" />
+    </joint>
+    <link name="${name_prefix}gps">
       <visual>
         <geometry>

Commit message: nav2 sim

File: src/igvc/description/ackermann_ac.urdf (robot description, URDF)
Before this commit: robot sarah5, 6 links, 5 joints
Joints:
- joint footprint_joint: type None -> fixed

File: src/igvc/description/ackermann_gz.urdf (robot description, URDF)
Before this commit: robot sarah6, 5 links, 4 joints
Links:
- added link base_footprint
Joints:
- added joint footprint_joint: type fixed, parent base_link, child base_footprint, origin xyz=0.0 0.0 -0.1014 rpy=0.0 0.0 0.0
- joint chassis_joint: origin xyz=${chassis_offset} -> xyz=-0.4575 0.0 0.1955 rpy=0.0 -0.0208 0.0
- joint diff_joint: origin xyz=-${track_width} 0 0 -> xyz=-0.815 0 0
- joint front_left_steering_joint: origin xyz=0 ${wheel_base/2} 0 -> xyz=0 ${wheel_base_f/2} 0
- joint front_right_steering_joint: origin xyz=0 -${wheel_base/2} 0 -> xyz=0 -${wheel_base_f/2} 0

File: src/igvc/description/macros/components.xacro (robot description, xacro)
@@ -260,17 +260,4 @@
       </visual>
     </link>
-    <!-- <gazebo reference="${name}">
-      <sensor name="imu" type="imu">
-        <pose>0 0 0 0 0 0</pose>
-        <always_on>true</always_on>
-        <update_rate>20</update_rate>
-        <visualize>true</visualize>
-        <topic>imu</topic>
-        <gz_frame_id>imu</gz_frame_id>
-        <plugin filename="libignition-gazebo-imu-system.so"
-          name="ignition::gazebo::systems::Imu">
-        </plugin>
-      </sensor>
-    </gazebo> -->
   </xacro:macro>
   <!--

File: src/igvc/description/macros/materials.xacro (robot description, xacro)
@@ -2,5 +2,5 @@
 <robot xmlns:xacro="http://www.ros.org/wiki/xacro">
     <material name="white">
-        <color rgba="1 1 1 0.1" />
+        <color rgba="1 1 1 0.8" />
     </material>
     <material name="black">
